File: shikisaku/shikisaku.kicad_pcb (KiCad board)
At the start: 2 copper layers, 0 parts

Commit message: layout footprints
Parts:
- added BT1: 3.6V, Connector_JST:JST_XH_S2B-XH-A_1x02_P2.50mm_Horizontal, F.Cu at (109.8, 100.7)
- added D1: LED_RGBA, akizuki:LED_OSTBMAZ2C1D, B.Cu at (129.2, 66.6)
- added D2: LED_RGBA, akizuki:LED_OSTBMAZ2C1D, B.Cu at (156.9, 89.2)
- added D3: LED_RGBA, akizuki:LED_OSTBMAZ2C1D, B.Cu at (134.3, 116.9)
- added D4: LED_RGBA, akizuki:LED_OSTBMAZ2C1D, B.Cu at (106.6, 94.3)
- added Q1: 2SC1815, Package_TO_SOT_THT:TO-92_Inline, F.Cu at (126.7, 110.8)
- added Q2: 2SC1815, Package_TO_SOT_THT:TO-92_Inline, F.Cu at (133.0, 110.8)
- added Q3: 2SC1815, Package_TO_SOT_THT:TO-92_Inline, F.Cu at (139.4, 110.8)
- added R1: 10k, Resistor_THT:R_Axial_DIN0207_L6.3mm_D2.5mm_P7.62mm_Horizontal, F.Cu at (112.7, 110.8)
- added R2: 10k, Resistor_THT:R_Axial_DIN0207_L6.3mm_D2.5mm_P7.62mm_Horizontal, F.Cu at (112.7, 114.6)
- added R3: 10k, Resistor_THT:R_Axial_DIN0207_L6.3mm_D2.5mm_P7.62mm_Horizontal, F.Cu at (112.7, 118.4)
- added RN1: 22, Resistor_SMD:R_Array_Convex_4x0603_1, F.Cu at (145.8, 111.2)
- added RN2: 22, Resistor_SMD:R_Array_Convex_4x0603_1, F.Cu at (152.1, 111.2)
- added RN3: 22, Resistor_SMD:R_Array_Convex_4x0603_1, F.Cu at (158.5, 111.2)
- added SW1: SW_Reset, Button_Switch_THT:SW_PUSH_1P1T_6x3.5mm_H4.3_APEM_MJTP1243, F.Cu at (114.5, 62.5)
- added SW2: SW_Push, Connector_JST:JST_XH_B2B-XH-A_1x02_P2.50mm_Vertical, F.Cu at (147.0, 65.1)
- added SW3: SW_SPST, Connector_JST:JST_XH_B2B-XH-A_1x02_P2.50mm_Vertical, F.Cu at (119.0, 103.2)
- added U1: ProMicro, promicro:ProMicro-EnforcedTop, F.Cu at (119.0, 77.8)
- added U2: MMC5603, Adafruit:MMC5603, B.Cu at (133.0, 90.5)
- added U3: HC-SR04, Connector_JST:JST_XH_B4B-XH-A_1x04_P2.50mm_Vertical, B.Cu at (139.5, 82.9)
- added U4: HC-SR04, Connector_JST:JST_XH_B4B-XH-A_1x04_P2.50mm_Vertical, B.Cu at (139.5, 74.0)
- added U5: XCL103, akizuki:XCL103, F.Cu at (120.3, 94.3)
Other:
- board outline added: 63.5 x 63.5 mm

Commit message: add mounting holes
Parts:
- added REF**: MountingHole_3.2mm_M3, MountingHole:MountingHole_3.2mm_M3, F.Cu at (104.0, 119.5)
- added REF**: MountingHole_3.2mm_M3, MountingHole:MountingHole_3.2mm_M3, F.Cu at (104.0, 64.0)
- added REF**: MountingHole_3.2mm_M3, MountingHole:MountingHole_3.2mm_M3, F.Cu at (159.5, 119.5)
- added REF**: MountingHole_3.2mm_M3, MountingHole:MountingHole_3.2mm_M3, F.Cu at (159.5, 64.0)
Changed lines of the file:
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@@
     )
     (pad_to_mask_clearance 0)
-    (grid_origin 100 60)
+    (grid_origin 100 123.5)
     (pcbplotparams
       (layerselection 0x00010fc_ffffffff)
@@
     (property "ki_keywords" "batt voltage-source cell")
     (attr through_hole)
-    (fp_text reference "BT1" (at 1.25 -3.5 90) (layer "F.SilkS")
+    (fp_text reference "BT1" (at 6.84 2.8 -180) (layer "F.SilkS")
         (effects (font (size 1 1) (thickness 0.153)))
     )
@@
     )
   )
+  (footprint "MountingHole:MountingHole_3.2mm_M3" (layer "F.Cu")
+    (at 104 119.5)
+    (descr "Mounting Hole 3.2mm, no annular, M3")
+    (tags "mounting hole 3.2mm no annular m3")
+    (attr exclude_from_pos_files exclude_from_bom)
+    (fp_text reference "REF**" (at 0 -4.2) (layer "F.SilkS") hide
+        (effects (font (size 1 1) (thickness 0.15)))
+    )
+    (fp_text value "MountingHole_3.2mm_M3" (at 0 4.2) (layer "F.Fab") hide
+        (effects (font (size 1 1) (thickness 0.15)))
+    )
+    (fp_circle (center 0 0) (end 3.2 0)
+      (stroke (width 0.15) (type solid)) (fill none) (layer "Cmts.User"))
+    (fp_circle (center 0 0) (end 3.45 0)
+      (stroke (width 0.05) (type solid)) (fill none) (layer "F.CrtYd"))
+    (pad "" np_thru_hole circle (at 0 0) (size 3.2 3.2) (drill 3.2) (layers "F&B.Cu" "*.Mask"))
+  )
   (footprint "Resistor_SMD:R_Array_Convex_4x0603_1" (layer "F.Cu")
     (at 145.79 111.22 90)
@@
     )
   )
+  (footprint "MountingHole:MountingHole_3.2mm_M3" (layer "F.Cu")
+    (at 104 64)
+    (descr "Mounting Hole 3.2mm, no annular, M3")
+    (tags "mounting hole 3.2mm no annular m3")
+    (attr exclude_from_pos_files exclude_from_bom)
+    (fp_text reference "REF**" (at 0 -4.2) (layer "F.SilkS") hide
+        (effects (font (size 1 1) (thickness 0.15)))
+    )
+    (fp_text value "MountingHole_3.2mm_M3" (at 0 4.2) (layer "F.Fab") hide
+        (effects (font (size 1 1) (thickness 0.15)))
+    )
+    (fp_circle (center 0 0) (end 3.2 0)
+      (stroke (width 0.15) (type solid)) (fill none) (layer "Cmts.User"))
+    (fp_circle (center 0 0) (end 3.45 0)
+      (stroke (width 0.05) (type solid)) (fill none) (layer "F.CrtYd"))
+    (pad "" np_thru_hole circle (at 0 0) (size 3.2 3.2) (drill 3.2) (layers "*.Cu" "*.Mask"))
+  )
   (footprint "Package_TO_SOT_THT:TO-92_Inline" (layer "F.Cu")
     (at 139.37 110.8 180)
@@
     )
   )
+  (footprint "MountingHole:MountingHole_3.2mm_M3" (layer "F.Cu")
+    (at 159.5 119.5)
+    (descr "Mounting Hole 3.2mm, no annular, M3")
+    (tags "mounting hole 3.2mm no annular m3")
+    (attr exclude_from_pos_files exclude_from_bom)
+    (fp_text reference "REF**" (at 0 -4.2) (layer "F.SilkS") hide
+        (effects (font (size 1 1) (thickness 0.15)))
+    )
+    (fp_text value "MountingHole_3.2mm_M3" (at 0 4.2) (layer "F.Fab") hide
+        (effects (font (size 1 1) (thickness 0.15)))
+    )
+    (fp_circle (center 0 0) (end 3.2 0)
+      (stroke (width 0.15) (type solid)) (fill none) (layer "Cmts.User"))
+    (fp_circle (center 0 0) (end 3.45 0)
+      (stroke (width 0.05) (type solid)) (fill none) (layer "F.CrtYd"))
+    (pad "" np_thru_hole circle (at 0 0) (size 3.2 3.2) (drill 3.2) (layers "F&B.Cu" "*.Mask"))
+  )
   (footprint "Resistor_THT:R_Axial_DIN0207_L6.3mm_D2.5mm_P7.62mm_Horizontal" (layer "F.Cu")
     (at 112.7 114.61)
@@
       (rotate (xyz 0 0 0))
     )
+  )
+  (footprint "MountingHole:MountingHole_3.2mm_M3" (layer "F.Cu")
+    (at 159.5 64)
+    (descr "Mounting Hole 3.2mm, no annular, M3")
+    (tags "mounting hole 3.2mm no annular m3")
+    (attr exclude_from_pos_files exclude_from_bom)
+    (fp_text reference "REF**" (at 0 -4.2) (layer "F.SilkS") hide
+        (effects (font (size 1 1) (thickness 0.15)))
+    )
+    (fp_text value "MountingHole_3.2mm_M3" (at 0 4.2) (layer "F.Fab") hide
+        (effects (font (size 1 1) (thickness 0.15)))
+    )
+    (fp_circle (center 0 0) (end 3.2 0)
+      (stroke (width 0.15) (type solid)) (fill none) (layer "Cmts.User"))
+    (fp_circle (center 0 0) (end 3.45 0)
+      (stroke (width 0.05) (type solid)) (fill none) (layer "F.CrtYd"))
+    (pad "" np_thru_hole circle (at 0 0) (size 3.2 3.2) (drill 3.2) (layers "*.Cu" "*.Mask"))
   )
   (footprint "Connector_JST:JST_XH_B4B-XH-A_1x04_P2.50mm_Vertical" (layer "B.Cu")
@@
       (net 9 "Net-(D2-RK)") (pinfunction "RK") (pintype "passive"))
   )
+  (gr_line (start 101 68) (end 108 68)
+    (stroke (width 0.15) (type default)) (layer "F.SilkS"))
+  (gr_line (start 108 68) (end 108 61)
+    (stroke (width 0.15) (type default)) (layer "F.SilkS"))
+  (gr_line (start 108 115.5) (end 108 122.5)
+    (stroke (width 0.15) (type default)) (layer "F.SilkS"))
+  (gr_line (start 162.5 115.5) (end 155.5 115.5)
+    (stroke (width 0.15) (type default)) (layer "F.SilkS"))
+  (gr_line (start 155.5 115.5) (end 155.5 122.5)
+    (stroke (width 0.15) (type default)) (layer "F.SilkS"))
+  (gr_line (start 101 115.5) (end 108 115.5)
+    (stroke (width 0.15) (type default)) (layer "F.SilkS"))
+  (gr_line (start 155.5 61) (end 155.5 68)
+    (stroke (width 0.15) (type default)) (layer "F.SilkS"))
+  (gr_line (start 155.5 68) (end 162.5 68)
+    (stroke (width 0.15) (type default)) (layer "F.SilkS"))
   (gr_rect (start 100 123.5) (end 163.5 60)
     (stroke (width 0.1) (type default)) (fill none) (layer "Edge.Cuts"))
-  (zone (net 0) (net_name "") (layers "F&B.Cu" "*.SilkS" "*.Mask" "Edge.Cuts") (name "Spacer") (hatch edge 0.5)
-    (connect_pads (clearance 0))
-    (min_thickness 0.25) (filled_areas_thickness no)
-    (keepout (tracks not_allowed) (vias not_allowed) (pads not_allowed) (copperpour allowed) (footprints not_allowed))
-    (fill (thermal_gap 0.5) (thermal_bridge_width 0.5))
-    (polygon
-      (pts
-        (xy 100 60)
-        (xy 100 68)
-        (xy 108 68)
-        (xy 108 60)
-      )
-    )
-  )
-  (zone (net 0) (net_name "") (layers "F&B.Cu" "*.SilkS" "*.Mask" "Edge.Cuts") (name "Spacer") (hatch edge 0.5)
-    (connect_pads (clearance 0))
-    (min_thickness 0.25) (filled_areas_thickness no)
-    (keepout (tracks not_allowed) (vias not_allowed) (pads not_allowed) (copperpour allowed) (footprints not_allowed))
-    (fill (thermal_gap 0.5) (thermal_bridge_width 0.5))
-    (polygon
-      (pts
-        (xy 100 123.5)
-        (xy 100 115.5)
-        (xy 108 115.5)
-        (xy 108 123.5)
-      )
-    )
-  )
-  (zone (net 0) (net_name "") (layers "F&B.Cu" "*.SilkS" "*.Mask" "Edge.Cuts") (name "Spacer") (hatch edge 0.5)
-    (connect_pads (clearance 0))
-    (min_thickness 0.25) (filled_areas_thickness no)
-    (keepout (tracks not_allowed) (vias not_allowed) (pads not_allowed) (copperpour allowed) (footprints not_allowed))
-    (fill (thermal_gap 0.5) (thermal_bridge_width 0.5))
-    (polygon
-      (pts
-        (xy 163.5 123.5)
-        (xy 155.5 123.5)
-        (xy 155.5 115.5)
-        (xy 163.5 115.5)
-      )
-    )
-  )
-  (zone (net 0) (net_name "") (layers "F&B.Cu" "*.SilkS" "*.Mask" "Edge.Cuts") (name "Spacer") (hatch edge 0.5)
-    (connect_pads (clearance 0))
-    (min_thickness 0.25) (filled_areas_thickness no)
-    (keepout (tracks not_allowed) (vias not_allowed) (pads not_allowed) (copperpour allowed) (footprints not_allowed))
-    (fill (thermal_gap 0.5) (thermal_bridge_width 0.5))
-    (polygon
-      (pts
-        (xy 163.5 60)
-        (xy 163.5 68)
-        (xy 155.5 68)
-        (xy 155.5 60)
-      )
-    )
-  )
 )
