File: shikisaku/shikisaku.kicad_pcb (KiCad board)
At the start: 2 copper layers, 63.5 x 63.5 mm, 26 parts, among them Q1 2SC1815, Q2 2SC1815, Q3 2SC1815, SW1 SW_Reset, SW2 SW_Push, SW3 SW_SPST, U1 ProMicro, U2 MMC5603, U3 HC-SR04, U4 HC-SR04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

Commit message: 配線(仮)
Parts:
- moved U4 11.8 mm to (149.0, 81.0), turned to 90 degrees
- moved U3 1.93 mm to (140.0, 81.0), turned to 90 degrees
Routing:
- net GND: track 0.00 -> 197.3 mm, vias 0 -> 3
- net VCC: track 0.00 -> 144.8 mm, vias 0 -> 1
- net Net-(D4-BK): track 0.00 -> 71.5 mm, vias 0 -> 1
- net Net-(D4-GK): track 0.00 -> 63.6 mm, vias 0 -> 1
- net LED_B: track 0.00 -> 57.6 mm
- net Net-(D1-GK): track 0.00 -> 56.8 mm
- net Net-(D1-RK): track 0.00 -> 55.2 mm
- net Net-(D4-RK): track 0.00 -> 54.1 mm, vias 0 -> 1
- net Net-(D1-BK): track 0.00 -> 53.3 mm
- net Net-(D2-RK): track 0.00 -> 38.3 mm
- net LED_G: track 0.00 -> 37.6 mm
- net Net-(D3-GK): track 0.00 -> 36.3 mm, vias 0 -> 2
- net Net-(D3-BK): track 0.00 -> 35.4 mm, vias 0 -> 2
- net SDA: track 0.00 -> 32.2 mm
- net LED_R: track 0.00 -> 30.3 mm
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
Commit message: use SK6812MINI-E
Changed lines of the file:
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@@
   (gr_line (start 155.5 68) (end 162.5 68)
     (stroke (width 0.15) (type default)) (layer "F.SilkS"))
-  (gr_rect (start 100 123.5) (end 163.5 60)
+  (gr_rect (start 100 60) (end 163.5 123.5)
     (stroke (width 0.1) (type default)) (fill none) (layer "Edge.Cuts"))
   (segment (start 109.8 100.66) (end 109.8 97.22) (width 0.25) (layer "F.Cu") (net 1))

Commit message: 配置
Parts:
- removed Q1, Q2, Q3: 2SC1815, Package_TO_SOT_THT:TO-92_Inline
- removed R2, R3: 10k, Resistor_THT:R_Axial_DIN0207_L6.3mm_D2.5mm_P7.62mm_Horizontal
- removed REF** (x4): MountingHole_3.2mm_M3, MountingHole:MountingHole_3.2mm_M3
- removed RN1, RN2, RN3: 22, Resistor_SMD:R_Array_Convex_4x0603_1
- added C1: 4.7u, Capacitor_SMD:C_0805_2012Metric_Pad1.18x1.45mm_HandSolder, B.Cu at (120.1, 87.9)
- added D5: SK6812MINI-E, LED_SMD:LED_SK6812MINI-E, F.Cu at (162.7, 78.6)
- added D6: SK6812MINI-E, LED_SMD:LED_SK6812MINI-E, F.Cu at (139.0, 60.8)
- added D7: SK6812MINI-E, LED_SMD:LED_SK6812MINI-E, F.Cu at (118.6, 60.8)
- added D8: SK6812MINI-E, LED_SMD:LED_SK6812MINI-E, F.Cu at (100.8, 84.5)
- added H1: MountingHole, MountingHole:MountingHole_3.2mm_M3, F.Cu at (104.0, 64.0)
- added H2: MountingHole, MountingHole:MountingHole_3.2mm_M3, F.Cu at (159.5, 64.0)
- added H3: MountingHole, MountingHole:MountingHole_3.2mm_M3, F.Cu at (159.5, 119.5)
- added H4: MountingHole, MountingHole:MountingHole_3.2mm_M3, F.Cu at (104.0, 119.5)
- D1, D2, D3, D4: value LED_RGBA -> SK6812MINI-E; footprint akizuki:LED_OSTBMAZ2C1D -> LED_SMD:LED_SK6812MINI-E; moved to F.Cu
- R1: value 10k -> 220
- moved D4 56.3 mm to (162.7, 99.0)
- moved D1 47.7 mm to (100.8, 104.9), turned to 90 degrees
- moved D2 46.6 mm to (124.5, 122.7), turned to 180 degrees
- moved SW2 16.5 mm to (130.5, 63.8), turned to 0 degrees
- moved R1 13.7 mm to (105.1, 99.4)
- moved D3 12.0 mm to (144.9, 122.7), turned to 180 degrees
- moved BT1 10.2 mm to (109.8, 90.5)
- moved U5 5.43 mm to (116.5, 98.1), turned to 90 degrees
- moved SW1 3.70 mm to (117.2, 65.1), turned to 180 degrees
- moved U2 1.27 mm to (131.8, 90.5)
- moved SW3 1.23 mm to (117.8, 103.2), turned to 0 degrees
- moved U3 0.47 mm to (140.0, 81.5)
- moved U4 0.47 mm to (149.0, 81.5)
Connections:
- D1 pad 1: VCC -> +5V
- D1 pad 2: Net-(D1-BK) -> Net-(D1-DOUT)
- D1 pad 3: Net-(D1-GK) -> GND
- D1 pad 4: Net-(D1-RK) -> Net-(D1-DIN)
- D2 pad 1: VCC -> +5V
- D2 pad 2: Net-(D2-BK) -> Net-(D2-DOUT)
- D2 pad 3: Net-(D2-GK) -> GND
- D2 pad 4: Net-(D2-RK) -> Net-(D1-DOUT)
- D3 pad 1: VCC -> +5V
- D3 pad 2: Net-(D3-BK) -> Net-(D3-DOUT)
- D3 pad 3: Net-(D3-GK) -> GND
- D3 pad 4: Net-(D3-RK) -> Net-(D2-DOUT)
- D4 pad 1: VCC -> +5V
- D4 pad 3: Net-(D4-GK) -> GND
- D4 pad 4: Net-(D4-RK) -> Net-(D3-DOUT)
- R1 pad 1: LED_R -> LED
- R1 pad 2: Net-(Q1-B) -> Net-(D1-DIN)
- U1 pad 1: unconnected-(U1-TX-Pad1) -> LED
- U1 pad 12: LED_G -> unconnected-(U1-B5-Pad12)
- U1 pad 13: LED_B -> unconnected-(U1-B6-Pad13)
- U1 pad 8: LED_R -> unconnected-(U1-C6-Pad8)
Routing:
- net GND: track 197.3 -> 0.00 mm, vias 3 -> 0
- net VCC: track 144.8 -> 0.00 mm, vias 1 -> 0
- net Net-(D4-DOUT): track 71.5 -> 0.00 mm, vias 1 -> 0
- net Net-(D4-GK): track 63.6 -> 0.00 mm, vias 1 -> 0
- net LED_B: track 57.6 -> 0.00 mm
- net Net-(D1-GK): track 56.8 -> 0.00 mm
- net Net-(D1-RK): track 55.2 -> 0.00 mm
- net Net-(D4-RK): track 54.1 -> 0.00 mm, vias 1 -> 0
- net Net-(D1-BK): track 53.3 -> 0.00 mm
- net Net-(D2-RK): track 38.3 -> 0.00 mm
- net LED_G: track 37.6 -> 0.00 mm
- net Net-(D3-GK): track 36.3 -> 0.00 mm, vias 2 -> 0
- net Net-(D3-BK): track 35.4 -> 0.00 mm, vias 2 -> 0
- net SDA: track 32.2 -> 0.00 mm
- net LED_R: track 30.3 -> 0.00 mm
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
Commit message: 配線完了
Parts:
- C1: moved to F.Cu
- D1, D2, D3, D4, D5, D6, D7, D8: moved to B.Cu
- moved C1 18.3 mm to (112.7, 104.7), turned to 90 degrees
- moved SW3 10.6 mm to (121.0, 93.0), turned to 180 degrees
- moved R1 7.62 mm to (112.7, 99.4), turned to 180 degrees
- moved U5 4.45 mm to (121.0, 98.1), turned to -90 degrees
- moved D1 1.63 mm to (102.3, 105.5)
- moved D2 1.63 mm to (123.9, 121.2)
- moved D4 1.63 mm to (161.2, 99.6)
- moved D5 1.63 mm to (161.2, 78.0)
- moved D7 1.63 mm to (118.0, 62.3)
- moved D8 1.63 mm to (102.3, 83.9)
- moved D3 1.63 mm to (145.5, 121.2)
- moved D6 1.63 mm to (139.6, 62.3)
- moved SW1 0.71 mm to (116.5, 65.1)
- moved U4 0.11 mm to (148.9, 81.5)
Routing:
- net GND: track 0.00 -> 292.3 mm, vias 0 -> 7
- net +5V: track 0.00 -> 209.8 mm, vias 0 -> 2
- net VCC: track 0.00 -> 63.2 mm
- net SDA: track 0.00 -> 34.1 mm
- net SCL: track 0.00 -> 27.8 mm
- net TRIG_V: track 0.00 -> 26.9 mm
- net Net-(D7-DOUT): track 0.00 -> 26.5 mm
- net +BATT: track 0.00 -> 24.6 mm
- net Net-(D1-DOUT): track 0.00 -> 23.9 mm
- net Net-(D5-DOUT): track 0.00 -> 23.9 mm
- net Net-(D3-DOUT): track 0.00 -> 23.9 mm
- net TRIG_H: track 0.00 -> 22.5 mm
- net ECHO_V: track 0.00 -> 22.4 mm
- net LED: track 0.00 -> 20.4 mm
- net ECHO_H: track 0.00 -> 18.0 mm
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- added copper zone on B.Cu, net GND
- added copper zone on F.Cu, net GND

Commit message: complete and output Gerber
Parts:
- added G***: LOGO, LOGO, F.Cu at (131.8, 112.7)
- added REF**: Shikisaku, Logo:Shikisaku, B.Cu at (131.8, 112.7)
- renumbered BT1 to BATT, SW2 to SW_KEY, SW3 to SW_POWER, SW1 to SW_RST, U3 to U3_H, U4 to U4_V
Routing:
- net SDA: track 34.1 -> 33.6 mm
Other:
- board text added: "JLCJLCJLCJLC"
- board text added: "Shikisaku designed by object1037"
