File: shikisaku/shikisaku.kicad_sch (KiCad schematic)
At the start: 19 parts, among them SW1 SW_Reset, SW2 SW_Push, SW3 SW_SPST, U1 ProMicro, U2 MMC5603, U3 HC-SR04, U4 HC-SR04, U5 XCL103

Commit message: 配置
Parts:
- added H1, H2, H3, H4: MountingHole, MountingHole:MountingHole_3.2mm_M3, symbol Mechanical:MountingHole
Other:
- note added: "Holes"
Changed lines of the file:
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@@
+    (fill (type none))
+  )
+  (rectangle (start 27.94 143.51) (end 71.12 163.83)
+    (stroke (width 0) (type dash))
     (fill (type none))
   )
@@
   )
   (text "Power" (at 29.21 74.93 0)
+    (effects (font (size 1.905 1.905)) (justify left bottom))
+  )
+  (text "Holes" (at 29.21 162.56 0)
     (effects (font (size 1.905 1.905)) (justify left bottom))
   )
@@
     )
   )
+  (symbol (lib_id "Mechanical:MountingHole") (at 33.02 154.94 0) (unit 1)
+    (in_bom yes) (on_board yes) (dnp no) (fields_autoplaced)
+    (property "Reference" "H2" (at 35.56 153.67 0)
+      (effects (font (size 1.27 1.27)) (justify left))
+    )
+    (property "Value" "MountingHole" (at 35.56 156.21 0)
+      (effects (font (size 1.27 1.27)) (justify left))
+    )
+    (property "Footprint" "MountingHole:MountingHole_3.2mm_M3" (at 33.02 154.94 0)
+      (effects (font (size 1.27 1.27)) hide)
+    )
+    (property "Datasheet" "~" (at 33.02 154.94 0)
+      (effects (font (size 1.27 1.27)) hide)
+    )
+    (instances
+      (project "shikisaku"
+        (path "/a06eb673-4587-4fcb-8c7b-235222103f86"
+          (reference "H2") (unit 1)
+        )
+      )
+    )
+  )
   (symbol (lib_id "power:GND") (at 92.71 124.46 0) (unit 1)
     (in_bom yes) (on_board yes) (dnp no)
@@
     )
   )
+  (symbol (lib_id "Mechanical:MountingHole") (at 33.02 148.59 0) (unit 1)
+    (in_bom yes) (on_board yes) (dnp no) (fields_autoplaced)
+    (property "Reference" "H1" (at 35.56 147.32 0)
+      (effects (font (size 1.27 1.27)) (justify left))
+    )
+    (property "Value" "MountingHole" (at 35.56 149.86 0)
+      (effects (font (size 1.27 1.27)) (justify left))
+    )
+    (property "Footprint" "MountingHole:MountingHole_3.2mm_M3" (at 33.02 148.59 0)
+      (effects (font (size 1.27 1.27)) hide)
+    )
+    (property "Datasheet" "~" (at 33.02 148.59 0)
+      (effects (font (size 1.27 1.27)) hide)
+    )
+    (instances
+      (project "shikisaku"
+        (path "/a06eb673-4587-4fcb-8c7b-235222103f86"
+          (reference "H1") (unit 1)
+        )
+      )
+    )
+  )
   (symbol (lib_id "power:GND") (at 115.57 63.5 0) (unit 1)
     (in_bom yes) (on_board yes) (dnp no) (fields_autoplaced)
@@
         (path "/a06eb673-4587-4fcb-8c7b-235222103f86"
           (reference "#PWR015") (unit 1)
+        )
+      )
+    )
+  )
+  (symbol (lib_id "Mechanical:MountingHole") (at 52.07 148.59 0) (unit 1)
+    (in_bom yes) (on_board yes) (dnp no) (fields_autoplaced)
+    (property "Reference" "H3" (at 54.61 147.32 0)
+      (effects (font (size 1.27 1.27)) (justify left))
+    )
+    (property "Value" "MountingHole" (at 54.61 149.86 0)
+      (effects (font (size 1.27 1.27)) (justify left))
+    )
+    (property "Footprint" "MountingHole:MountingHole_3.2mm_M3" (at 52.07 148.59 0)
+      (effects (font (size 1.27 1.27)) hide)
+    )
+    (property "Datasheet" "~" (at 52.07 148.59 0)
+      (effects (font (size 1.27 1.27)) hide)
+    )
+    (instances
+      (project "shikisaku"
+        (path "/a06eb673-4587-4fcb-8c7b-235222103f86"
+          (reference "H3") (unit 1)
         )
       )
@@
         )
       )
+    )
+  )
+  (symbol (lib_id "Mechanical:MountingHole") (at 52.07 154.94 0) (unit 1)
+    (in_bom yes) (on_board yes) (dnp no) (fields_autoplaced)
+    (property "Reference" "H4" (at 54.61 153.67 0)
+      (effects (font (size 1.27 1.27)) (justify left))
+    )
+    (property "Value" "MountingHole" (at 54.61 156.21 0)
+      (effects (font (size 1.27 1.27)) (justify left))
+    )
+    (property "Footprint" "MountingHole:MountingHole_3.2mm_M3" (at 52.07 154.94 0)
+      (effects (font (size 1.27 1.27)) hide)
+    )
+    (property "Datasheet" "~" (at 52.07 154.94 0)
+      (effects (font (size 1.27 1.27)) hide)
+    )
+    (instances
+      (project "shikisaku"
+        (path "/a06eb673-4587-4fcb-8c7b-235222103f86"
+          (reference "H4") (unit 1)
+        )
+      )
